File: ADA4898_LNA.kicad_sch (KiCad schematic)
At the start: 72 parts, among them J101 CONN_01X01, J102 CONN_01X01, J103 CONN_01X01, J104 CONN_01X01, P101 BNC, P102 SMA, P103 CONN_02X04, P104 HI-BW_SELECT, P105 BNC, P106 CONN_02X04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

Commit message: add notes
Other:
- note added: "+6 VDC"
- note added: "-6 VDC"
