File: LNA_PSU.kicad_sch (KiCad schematic)
At the start: 24 parts, among them J1201 CONN_01X03, J1202 HEATSINK, J1203 HEATSINK, T1201 CM-CHOKE, T1202 CM-CHOKE, U1201 LT1963A, U1202 LT3015

Commit message: add notes
Other:
- note added: "+6 VDC"
- note added: "-6 VDC"
Changed lines of the file:
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@@
     (stroke (width 0) (type default) (color 0 0 0 0))
+  )
+  (text "+6 VDC" (at 199.39 31.75 0)
+    (effects (font (size 1.27 1.27)) (justify left bottom))
+  )
+  (text "-6 VDC" (at 199.39 67.31 0)
+    (effects (font (size 1.27 1.27)) (justify left bottom))
   )
   (label "GND_in" (at 39.37 41.91 0)
